File: pcb/d70-buddy/d70-buddy.kicad_pcb (KiCad board)
At the start: 2 copper layers, 0 parts

Commit message: more pcb stuff
Parts:
- added C1: 10µF, Capacitor_SMD:C_0805_2012Metric, B.Cu at (85.0, 107.5)
- added C10: 4.7µF, Capacitor_SMD:C_0805_2012Metric, B.Cu at (69.6, 109.7)
- added C3: 4.7µF, Capacitor_SMD:C_0805_2012Metric, B.Cu at (90.2, 112.0)
- added C4: 4.7µF, Capacitor_SMD:C_0805_2012Metric, B.Cu at (85.0, 111.6)
- added C5: 10µF, Capacitor_SMD:C_0805_2012Metric, B.Cu at (90.2, 115.0)
- added C6: 4.7µF, Capacitor_SMD:C_0805_2012Metric, B.Cu at (59.4, 104.4)
- added C7: 4.7µF, Capacitor_SMD:C_0805_2012Metric, B.Cu at (85.8, 114.7)
- added C8: 1.0µF, Capacitor_SMD:C_0603_1608Metric, B.Cu at (95.0, 110.0)
- added C9: 1.0µF, Capacitor_SMD:C_0603_1608Metric, B.Cu at (90.4, 117.8)
- added H1: ELW2106AA, lib:MOLEX_503480-1400, F.Cu at (170.0, 93.0)
- added J1: Conn_02x11_Top_Bottom, Connector_PinHeader_2.54mm:PinHeader_2x11_P2.54mm_Vertical, F.Cu at (231.1, 107.0)
- added L1: 10µH, Inductor_SMD:L_1812_4532Metric, B.Cu at (79.0, 112.0)
- added Q1: 2N2219, Package_TO_SOT_SMD:TSOT-23, B.Cu at (47.0, 107.0)
- added R1: 1K, Resistor_SMD:R_0402_1005Metric, B.Cu at (74.0, 114.0)
- added R3: 1.37M, Resistor_SMD:R_0402_1005Metric, B.Cu at (80.0, 116.0)
- added R4: 71.5k, Resistor_SMD:R_0402_1005Metric, B.Cu at (87.0, 117.5)
- added R5: 100, Resistor_SMD:R_0402_1005Metric, B.Cu at (60.1, 106.9)
- added SW1: SW_Push_LED, lib:SW_PUSH_LED_6mm_H7.3mm, F.Cu at (34.0, 110.0)
- added TP1: TestPoint, TestPoint:TestPoint_Pad_D1.5mm, F.Cu at (69.1, 68.7)
- added TP2: TestPoint, TestPoint:TestPoint_Pad_D1.5mm, F.Cu at (95.1, 50.1)
- added TP3: TestPoint, TestPoint:TestPoint_Pad_D1.0mm, F.Cu at (68.9, 72.0)
- added TP4: TestPoint, TestPoint:TestPoint_Pad_D1.0mm, F.Cu at (78.5, 62.1)
- added TP5: TestPoint, TestPoint:TestPoint_Pad_D1.0mm, F.Cu at (82.5, 59.6)
- added TP6: TestPoint, TestPoint:TestPoint_Pad_D1.0mm, F.Cu at (90.4, 52.8)
- added TP7: TestPoint, TestPoint:TestPoint_Pad_D1.0mm, F.Cu at (72.4, 68.4)
- added U1: TLV61046ADB, Package_TO_SOT_SMD:SOT-23-6, B.Cu at (91.0, 107.0)
- added U2: TLV70228_SOT23-5, Package_TO_SOT_SMD:SOT-23-5, B.Cu at (78.9, 107.0)
Routing:
- added copper zone on B.Cu, net GND
Other:
- board outline added: 210 x 18 mm

Commit message: wip
Parts:
- removed C1, C5: 10µF, Capacitor_SMD:C_0805_2012Metric
- removed C10, C3, C4, C6, C7: 4.7µF, Capacitor_SMD:C_0805_2012Metric
- removed C8, C9: 1.0µF, Capacitor_SMD:C_0603_1608Metric
- removed H1: ELW2106AA, lib:MOLEX_503480-1400
- removed L1: 10µH, Inductor_SMD:L_1812_4532Metric
- removed Q1: 2N2219, Package_TO_SOT_SMD:TSOT-23
- removed TP1, TP2: TestPoint, TestPoint:TestPoint_Pad_D1.5mm
- removed TP3, TP4, TP5, TP6, TP7: TestPoint, TestPoint:TestPoint_Pad_D1.0mm
- removed U1: TLV61046ADB, Package_TO_SOT_SMD:SOT-23-6
- removed U2: TLV70228_SOT23-5, Package_TO_SOT_SMD:SOT-23-5
- added J2: Conn_02x04_Top_Bottom, lib:ELW2106AA, F.Cu at (154.4, 102.0)
- added R2: 150, Resistor_SMD:R_0402_1005Metric, F.Cu at (81.5, 114.5)
- added R6: 150, Resistor_SMD:R_0402_1005Metric, F.Cu at (214.4, 114.2)
- added R7: 150, Resistor_SMD:R_0402_1005Metric, F.Cu at (246.0, 114.0)
- added SW2: SW_Push_LED_GREEN, lib:SW_PUSH_LED_6mm_H7.3mm, F.Cu at (71.0, 107.8)
- added SW3: SW_Push_LED_BLUE, lib:SW_PUSH_LED_6mm_H7.3mm, F.Cu at (87.0, 107.8)
- added SW4: SW_Push_LED_WHITE, lib:SW_PUSH_LED_6mm_H7.3mm, F.Cu at (103.5, 107.8)
- added SW5: SW_Push_LED_RED, lib:SW_PUSH_LED_6mm_H7.3mm, F.Cu at (200.2, 107.8)
- added SW6: SW_Push_LED_WHITE, lib:SW_PUSH_LED_6mm_H7.3mm, F.Cu at (218.0, 107.8)
- added SW7: SW_Push_LED_GREEN, lib:SW_PUSH_LED_6mm_H7.3mm, F.Cu at (235.8, 107.8)
- J1: moved to B.Cu
- R1: value 1K -> 68; moved to F.Cu
- R3: value 1.37M -> 150; moved to F.Cu
- R4: value 71.5k -> 150; moved to F.Cu
- R5: value 100 -> 68; moved to F.Cu
- SW1: value SW_Push_LED -> SW_Push_LED_YELLOW
- moved R5 137.0 mm to (197.0, 114.1)
- moved J1 88.8 mm to (142.3, 109.7)
- moved R4 26.7 mm to (113.5, 114.5), turned to 0 degrees
- moved SW1 21.4 mm to (55.2, 107.8)
- moved R3 17.6 mm to (97.5, 114.5), turned to 0 degrees
- moved R1 8.51 mm to (65.5, 114.5), turned to 0 degrees
Connections:
- J1 pad 10: /BTN_2 -> /LED_1
- J1 pad 11: /BTN_3 -> /BTN_2
- J1 pad 12: /BTN_4 -> /LED_2
- J1 pad 13: /BTN_5 -> /BTN_3
- J1 pad 14: /BTN_6 -> /LED_3
- J1 pad 15: /BTN_7 -> /BTN_4
- J1 pad 16: /LED_1 -> /LED_4
- J1 pad 17: /LED_2 -> /BTN_5
- J1 pad 18: /LED_3 -> /LED_5
- J1 pad 19: /LED_4 -> /BTN_6
- J1 pad 2: GND -> /RST
- J1 pad 20: /LED_5 -> /LED_6
- J1 pad 21: /LED_6 -> /BTN_7
- J1 pad 3: +3V3 -> GND
- J1 pad 4: /~{OLED_CS} -> /D/C
- J1 pad 5: /CMD_DATA -> VCC
- J1 pad 6: /~{OLED_RST} -> /SCLK
- J1 pad 7: /SPI1_MOSI -> /CS
- J1 pad 8: /SPI1_SCLK -> /MOSI
- R1 pad 1: /LED_1 -> Net-(SW1-Pad4)
- R1 pad 2: Net-(Q1-Pad2) -> /LED_1
- R3 pad 1: +16V -> Net-(SW3-Pad4)
- R3 pad 2: Net-(R3-Pad2) -> /LED_3
- R4 pad 1: Net-(R3-Pad2) -> Net-(SW4-Pad4)
- R4 pad 2: GND -> /LED_4
- R5 pad 1: Net-(R5-Pad1) -> Net-(SW5-Pad4)
- R5 pad 2: +3V3 -> /LED_5
- SW1 pad 3: Net-(Q1-Pad3) -> GND
- SW1 pad 4: Net-(R5-Pad1) -> Net-(SW1-Pad4)
Routing:
- net /LED_1: track 0.00 -> 106.8 mm, vias 0 -> 1
- net /BTN_1: track 0.00 -> 103.6 mm, vias 0 -> 2
- net /BTN_2: track 0.00 -> 91.9 mm, vias 0 -> 1
- net /LED_7: track 0.00 -> 82.1 mm
- net /BTN_3: track 0.00 -> 80.4 mm, vias 0 -> 2
- net /LED_2: track 0.00 -> 78.7 mm, vias 0 -> 1
- net /LED_3: track 0.00 -> 78.1 mm
- net /BTN_7: track 0.00 -> 76.4 mm
- net /BTN_4: track 0.00 -> 61.5 mm, vias 0 -> 1
- net /BTN_6: track 0.00 -> 61.3 mm
- net /LED_6: track 0.00 -> 52.7 mm
- net /BTN_5: track 0.00 -> 47.5 mm
- net /LED_5: track 0.00 -> 37.7 mm
- net /CS: track 0.00 -> 31.0 mm
- net /MOSI: track 0.00 -> 29.5 mm
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- added copper zone on F.Cu, net GND
Other:
- board size 210 x 18 mm -> 210 x 17.9 mm

Commit message: wip
Routing:
- net /LED_4: track 0.00 -> 48.9 mm
Changed lines of the file:
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@@
       (effects (font (size 1 1) (thickness 0.15)))
+    )
+    (fp_text user "GND" (at -27.005 5.29) (layer "F.SilkS")
+      (effects (font (size 0.6 0.6) (thickness 0.25)))
+    )
+    (fp_text user "CS" (at -35.295 5.5) (layer "F.SilkS")
+      (effects (font (size 0.6 0.6) (thickness 0.25)))
+    )
+    (fp_text user "MOSI\n" (at -34.545 12.588205) (layer "F.SilkS")
+      (effects (font (size 0.6 0.6) (thickness 0.25)))
+    )
+    (fp_text user "SCLK\n" (at -34.545 10.088205) (layer "F.SilkS")
+      (effects (font (size 0.6 0.6) (thickness 0.25)))
+    )
+    (fp_text user "RST" (at -26.995 10) (layer "F.SilkS")
+      (effects (font (size 0.6 0.6) (thickness 0.25)))
     )
     (fp_text user "D/C\n" (at -34.795 7.7) (layer "F.SilkS")
       (effects (font (size 0.6 0.6) (thickness 0.25)))
     )
-    (fp_text user "MOSI\n" (at -34.545 12.588205) (layer "F.SilkS")
-      (effects (font (size 0.6 0.6) (thickness 0.25)))
-    )
     (fp_text user "VCC" (at -26.995 7.5) (layer "F.SilkS")
-      (effects (font (size 0.6 0.6) (thickness 0.25)))
-    )
-    (fp_text user "RST" (at -26.995 10) (layer "F.SilkS")
-      (effects (font (size 0.6 0.6) (thickness 0.25)))
-    )
-    (fp_text user "GND" (at -27.005 5.29) (layer "F.SilkS")
-      (effects (font (size 0.6 0.6) (thickness 0.25)))
-    )
-    (fp_text user "SCLK\n" (at -34.545 10.088205) (layer "F.SilkS")
-      (effects (font (size 0.6 0.6) (thickness 0.25)))
-    )
-    (fp_text user "CS" (at -35.295 5.5) (layer "F.SilkS")
       (effects (font (size 0.6 0.6) (thickness 0.25)))
     )
@@
     (fp_rect (start -38.5 -0.022144) (end 38.5 17.877856) (layer "F.SilkS") (width 0.12) (fill none))
     (fp_circle (center -35.73 2.75) (end -33.98 2.75) (layer "F.CrtYd") (width 0.05) (fill none))
+    (fp_circle (center 35.77 2.75) (end 37.52 2.75) (layer "F.CrtYd") (width 0.05) (fill none))
     (fp_circle (center 35.77 15.25) (end 37.52 15.25) (layer "F.CrtYd") (width 0.05) (fill none))
     (fp_circle (center -35.73 15.25) (end -33.98 15.25) (layer "F.CrtYd") (width 0.05) (fill none))
-    (fp_circle (center 35.77 2.75) (end 37.52 2.75) (layer "F.CrtYd") (width 0.05) (fill none))
+    (fp_line (start 38.52 4.95) (end 38.52 0) (layer "F.Fab") (width 0.1))
+    (fp_line (start -38.48 0) (end 38.52 0) (layer "F.Fab") (width 0.1))
+    (fp_line (start 36.02 11.95) (end 37.52 11.95) (layer "F.Fab") (width 0.1))
+    (fp_line (start 38.52 17.9) (end -38.48 17.9) (layer "F.Fab") (width 0.1))
     (fp_line (start 35.52 6.45) (end 35.52 11.45) (layer "F.Fab") (width 0.1))
-    (fp_line (start -38.48 0) (end 38.52 0) (layer "F.Fab") (width 0.1))
-    (fp_line (start 38.52 17.9) (end -38.48 17.9) (layer "F.Fab") (width 0.1))
     (fp_line (start 38.52 17.9) (end 38.52 12.95) (layer "F.Fab") (width 0.1))
     (fp_line (start 36.02 5.95) (end 37.52 5.95) (layer "F.Fab") (width 0.1))
     (fp_line (start -38.48 17.9) (end -38.48 0) (layer "F.Fab") (width 0.1))
-    (fp_line (start 36.02 11.95) (end 37.52 11.95) (layer "F.Fab") (width 0.1))
-    (fp_line (start 38.52 4.95) (end 38.52 0) (layer "F.Fab") (width 0.1))
     (fp_rect (start 33.02 17.822145) (end -27.98 0.077856) (layer "F.Fab") (width 0.15) (fill none))
     (fp_rect (start 26.52 16.287856) (end -26.52 1.537856) (layer "F.Fab") (width 0.15) (fill none))
-    (fp_arc (start 36.02 11.95) (mid 35.666447 11.803553) (end 35.52 11.45) (layer "F.Fab") (width 0.1))
-    (fp_arc (start 35.52 6.45) (mid 35.666447 6.096447) (end 36.02 5.95) (layer "F.Fab") (width 0.1))
     (fp_arc (start 38.52 4.95) (mid 38.227106 5.657106) (end 37.52 5.95) (layer "F.Fab") (width 0.1))
     (fp_arc (start 37.52 11.95) (mid 38.227106 12.242894) (end 38.52 12.95) (layer "F.Fab") (width 0.1))
+    (fp_arc (start 35.52 6.45) (mid 35.666447 6.096447) (end 36.02 5.95) (layer "F.Fab") (width 0.1))
+    (fp_arc (start 36.02 11.95) (mid 35.666447 11.803553) (end 35.52 11.45) (layer "F.Fab") (width 0.1))
+    (pad "" np_thru_hole circle (at 35.77 2.75 180) (size 3 3) (drill 2.2) (layers F&B.Cu *.Mask))
+    (pad "" np_thru_hole circle (at 35.77 15.25 180) (size 3 3) (drill 2.2) (layers F&B.Cu *.Mask))
     (pad "" np_thru_hole circle (at -35.73 2.75 180) (size 3 3) (drill 2.2) (layers F&B.Cu *.Mask))
-    (pad "" np_thru_hole circle (at 35.77 15.25 180) (size 3 3) (drill 2.2) (layers F&B.Cu *.Mask))
-    (pad "" np_thru_hole circle (at 35.77 2.75 180) (size 3 3) (drill 2.2) (layers F&B.Cu *.Mask))
     (pad "" np_thru_hole circle (at -35.73 15.25 180) (size 3 3) (drill 2.2) (layers F&B.Cu *.Mask))
     (pad "1" thru_hole rect (at -29.64 4.85) (size 1.7 1.7) (drill 1) (layers *.Cu *.Mask)
@@
   (segment (start 158.805 111) (end 161.3 111) (width 0.4) (layer "F.Cu") (net 22))
   (segment (start 120.79 108.39) (end 119.198 109.982) (width 0.4) (layer "F.Cu") (net 22))
+  (segment (start 157.07548 116.02452) (end 121.69952 116.02452) (width 0.4) (layer "F.Cu") (net 23))
+  (segment (start 158.2 114.9) (end 157.07548 116.02452) (width 0.4) (layer "F.Cu") (net 23))
+  (segment (start 114.31 114.2) (end 114.01 114.5) (width 0.4) (layer "F.Cu") (net 23))
+  (segment (start 158.2 114.145) (end 158.2 114.9) (width 0.4) (layer "F.Cu") (net 23))
+  (segment (start 121.69952 116.02452) (end 119.875 114.2) (width 0.4) (layer "F.Cu") (net 23))
+  (segment (start 119.875 114.2) (end 114.31 114.2) (width 0.4) (layer "F.Cu") (net 23))
+  (segment (start 160.08 112.265) (end 158.2 114.145) (width 0.4) (layer "F.Cu") (net 23))
   (segment (start 171.709926 110.87) (end 193.96 110.87) (width 0.4) (layer "F.Cu") (net 24))
   (segment (start 162.62 112.265) (end 164.469031 114.114031) (width 0.4) (layer "F.Cu") (net 24))

Commit message: Wip
Parts:
- removed J2: Conn_02x04_Top_Bottom, lib:ELW2106AA
- added H1: MountingHole_2.2mm_M2, MountingHole:MountingHole_2.2mm_M2, F.Cu at (51.0, 102.8)
- added H2: MountingHole_2.2mm_M2, MountingHole:MountingHole_2.2mm_M2, F.Cu at (51.0, 111.2)
- added H3: MountingHole_2.2mm_M2, MountingHole:MountingHole_2.2mm_M2, F.Cu at (257.0, 102.8)
- added H4: MountingHole_2.2mm_M2, MountingHole:MountingHole_2.2mm_M2, F.Cu at (257.0, 111.2)
- added Q1: MBT2222A, Package_TO_SOT_SMD:SOT-23, F.Cu at (68.0, 105.8)
- added Q2: MBT2222A, Package_TO_SOT_SMD:SOT-23, F.Cu at (84.0, 105.8)
- added Q3: MBT2222A, Package_TO_SOT_SMD:SOT-23, F.Cu at (98.8, 102.8)
- added Q4: MBT2222A, Package_TO_SOT_SMD:SOT-23, F.Cu at (98.7, 109.7)
- added Q5: MBT2222A, Package_TO_SOT_SMD:SOT-23, F.Cu at (199.1, 106.3)
- added Q6: MBT2222A, Package_TO_SOT_SMD:SOT-23, F.Cu at (219.7, 106.0)
- added Q7: MBT2222A, Package_TO_SOT_SMD:SOT-23, F.Cu at (239.2, 105.6)
- added R10: 51, Resistor_SMD:R_0402_1005Metric, F.Cu at (94.8, 112.8)
- added R11: 51, Resistor_SMD:R_0402_1005Metric, F.Cu at (109.5, 112.8)
- added R12: 51, Resistor_SMD:R_0402_1005Metric, F.Cu at (198.0, 110.8)
- added R13: 51, Resistor_SMD:R_0402_1005Metric, F.Cu at (217.2, 110.2)
- added R14: 51, Resistor_SMD:R_0402_1005Metric, F.Cu at (237.9, 109.6)
- added R8: 51, Resistor_SMD:R_0402_1005Metric, F.Cu at (67.3, 111.2)
- added R9: 51, Resistor_SMD:R_0402_1005Metric, F.Cu at (83.2, 111.6)
- added U1: SSD1312_I2C_128x64, OLED SSD1312 KiCAD:OLED_SSD1312_I2C_0.96_No_Mounting_Holes, F.Cu at (133.4, 108.0)
- added U2: SSD1312_I2C_128x64, OLED SSD1312 KiCAD:OLED_SSD1312_I2C_0.96_No_Mounting_Holes, F.Cu at (174.6, 106.0)
- J1: value Conn_02x11_Top_Bottom -> Conn_02x12_Top_Bottom; footprint Connector_PinHeader_2.54mm:PinHeader_2x11_P2.54mm_Vertical -> Connector_PinHeader_2.54mm:PinHeader_2x12_P2.54mm_Vertical
- R1, R5: value 68 -> 25000; footprint Resistor_SMD:R_0402_1005Metric -> Resistor_SMD:R_0201_0603Metric
- R2, R3, R4, R6, R7: value 150 -> 25000; footprint Resistor_SMD:R_0402_1005Metric -> Resistor_SMD:R_0201_0603Metric
- SW2, SW7: value SW_Push_LED_GREEN -> SW_Push_LED_YELLOW
- SW3: value SW_Push_LED_BLUE -> SW_Push_LED_YELLOW
- SW4, SW6: value SW_Push_LED_WHITE -> SW_Push_LED_YELLOW
- SW5: value SW_Push_LED_RED -> SW_Push_LED_YELLOW
- moved R3 13.9 mm to (101.8, 101.2)
- moved R4 11.9 mm to (101.8, 112.5)
- moved SW7 11.0 mm to (246.8, 107.0)
- moved SW6 8.88 mm to (226.9, 107.0)
- moved R7 6.98 mm to (240.3, 109.9)
- moved R6 6.91 mm to (220.4, 110.8)
- moved SW5 6.80 mm to (207.0, 107.0)
- moved SW1 5.31 mm to (60.5, 107.0)
- moved SW2 5.06 mm to (76.0, 107.0)
- moved R1 4.88 mm to (68.9, 111.0), turned to -90 degrees
- moved R2 4.68 mm to (85.0, 111.3), turned to -90 degrees
- moved J1 4.60 mm to (140.0, 105.7)
- moved SW3 4.57 mm to (91.5, 107.0)
- moved R5 4.50 mm to (200.1, 110.8)
- moved SW4 3.54 mm to (107.0, 107.0)
Connections:
- J1 pad 10: /LED_1 -> /BTN_4
- J1 pad 11: /BTN_2 -> /LED_1
- J1 pad 12: /LED_2 -> /BTN_3
- J1 pad 13: /BTN_3 -> /BTN_2
- J1 pad 14: /LED_3 -> /BTN_5
- J1 pad 15: /BTN_4 -> /BTN_1
- J1 pad 16: /LED_4 -> /BTN_6
- J1 pad 17: /BTN_5 -> /LED_5
- J1 pad 18: /LED_5 -> /BTN_7
- J1 pad 19: /BTN_6 -> /LED_6
- J1 pad 2: /RST -> GND
- J1 pad 20: /LED_6 -> /SCL2
- J1 pad 21: /BTN_7 -> /LED_7
- J1 pad 22: /LED_7 -> /SDA2
- J1 pad 3: GND -> +3V3
- J1 pad 4: /D/C -> +5V
- J1 pad 5: VCC -> /SCL1
- J1 pad 6: /SCLK -> /LED_4
- J1 pad 7: /CS -> unconnected-(J1-Pad7)
- J1 pad 8: /MOSI -> /LED_3
- J1 pad 9: /BTN_1 -> /LED_2
- R1 pad 1: Net-(SW1-Pad4) -> Net-(Q1-Pad2)
- R2 pad 1: Net-(SW2-Pad4) -> Net-(R2-Pad1)
- R3 pad 1: Net-(SW3-Pad4) -> Net-(Q3-Pad2)
- R4 pad 1: Net-(SW4-Pad4) -> Net-(Q4-Pad2)
- R5 pad 1: Net-(SW5-Pad4) -> Net-(Q5-Pad2)
- R6 pad 1: Net-(SW6-Pad4) -> Net-(Q6-Pad2)
- R7 pad 1: Net-(SW7-Pad4) -> Net-(Q7-Pad2)
- SW1 pad 3: GND -> Net-(SW1-Pad3)
- SW2 pad 3: GND -> Net-(SW2-Pad3)
- SW2 pad 4: Net-(SW2-Pad4) -> Net-(R9-Pad1)
- SW3 pad 3: GND -> Net-(Q3-Pad3)
- SW3 pad 4: Net-(SW3-Pad4) -> Net-(R10-Pad1)
- SW4 pad 3: GND -> Net-(Q4-Pad3)
- SW4 pad 4: Net-(SW4-Pad4) -> Net-(R11-Pad1)
- SW5 pad 3: GND -> Net-(Q5-Pad3)
- SW5 pad 4: Net-(SW5-Pad4) -> Net-(R12-Pad1)
- SW6 pad 3: GND -> Net-(Q6-Pad3)
- SW6 pad 4: Net-(SW6-Pad4) -> Net-(R13-Pad1)
- SW7 pad 3: GND -> Net-(Q7-Pad3)
- SW7 pad 4: Net-(SW7-Pad4) -> Net-(R14-Pad1)
Routing:
- net +3V3: track 0.00 -> 184.9 mm
- net /SCL2: track 0.00 -> 32.3 mm
- net /SCL1: track 0.00 -> 31.3 mm
- net /CS: track 31.0 -> 0.00 mm
- net /SDA2: track 0.00 -> 29.8 mm
- net /MOSI: track 29.5 -> 0.00 mm
- net /LED_3: track 78.1 -> 49.7 mm, vias 0 -> 1
- net /SCLK: track 27.2 -> 0.00 mm
- net /BTN_7: track 76.4 -> 102.9 mm
- net /D/C: track 25.8 -> 0.00 mm
- net VCC: track 23.6 -> 0.00 mm
- net /BTN_6: track 61.3 -> 80.5 mm
- net /RST: track 18.3 -> 0.00 mm
- net /LED_1: track 106.8 -> 90.0 mm
- net Net-(R13-Pad1): track 0.00 -> 12.5 mm, vias 0 -> 1
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Other:
- board size 210 x 17.9 mm -> 212 x 14.5 mm

Commit message: Wip
Parts:
- Q1, Q2, Q3, Q4, Q5, Q6, Q7: footprint Package_TO_SOT_SMD:SOT-23 -> lib:MBT2222A
- R1, R2, R3, R4, R5, R6, R7: value 25000 -> 750; footprint Resistor_SMD:R_0201_0603Metric -> Resistor_SMD:R_0805_2012Metric_Pad1.20x1.40mm_HandSolder
- R10, R11, R12, R13, R14, R8, R9: footprint Resistor_SMD:R_0402_1005Metric -> Resistor_SMD:R_0805_2012Metric_Pad1.20x1.40mm_HandSolder
- moved R3 5.67 mm to (99.1, 106.2)
- moved R9 3.04 mm to (83.8, 108.6)
- moved R6 2.95 mm to (218.5, 108.5)
- moved R8 2.78 mm to (68.2, 108.6)
- moved R5 2.53 mm to (199.1, 108.4)
- moved R7 2.29 mm to (238.8, 108.2), turned to 180 degrees
- moved Q6 2.00 mm to (218.5, 104.4)
- moved Q5 1.87 mm to (199.1, 104.5)
- moved R14 1.62 mm to (238.8, 110.9)
- moved R13 1.52 mm to (218.5, 111.0), turned to 180 degrees
- moved R11 1.42 mm to (110.9, 112.8)
- moved Q1 1.38 mm to (68.3, 104.4)
- moved R4 1.36 mm to (103.1, 112.7)
- moved Q2 1.35 mm to (83.8, 104.4)
- moved R10 1.21 mm to (96.0, 112.7)
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Connections:
- J1 pad 7: unconnected-(J1-Pad7) -> /SDA1
- U1 pad 4: unconnected-(U1-Pad4) -> /SDA1
Routing:
- net +3V3: track 184.9 -> 237.9 mm, vias 0 -> 4
- net /SDA1: track 0.00 -> 36.0 mm
- net /LED_7: track 84.5 -> 76.9 mm
- net /BTN_3: track 68.5 -> 74.7 mm
- net /BTN_7: track 102.9 -> 97.8 mm
- net Net-(Q1-Pad2): track 4.01 -> 8.78 mm, vias 0 -> 2
- net Net-(R13-Pad1): track 12.5 -> 7.73 mm, vias 1 -> 0
- net /LED_5: track 43.7 -> 39.2 mm, vias 1 -> 0
- net /BTN_6: track 80.5 -> 76.0 mm
- net Net-(Q2-Pad2): track 4.34 -> 8.37 mm, vias 0 -> 2
- net /BTN_4: track 53.5 -> 49.4 mm
- net /LED_6: track 63.4 -> 59.6 mm
- net /BTN_1: track 106.7 -> 110.2 mm
- net Net-(R8-Pad1): track 6.70 -> 9.42 mm
- net Net-(R9-Pad1): track 7.20 -> 9.53 mm, vias 0 -> 1
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