File: pcb/d70-buddy-main-board/d70-buddy-main-board.kicad_pcb (KiCad board)
At the start: 2 copper layers, 100 x 100 mm, 12 parts, among them J1 PJ-327C-4A, J2 PJ-327C-4A, J3 Conn_02x12_Top_Bottom, U1 H11L1, U2 Pico

Commit message: Wip
Parts:
- removed R3: 68R, Resistor_SMD:R_0402_1005Metric
- added H1: MountingHole_3.2mm_M3_ISO7380_Pad, MountingHole:MountingHole_3.2mm_M3_ISO7380_Pad, F.Cu at (69.5, 50.5)
- added H2: MountingHole_3.2mm_M3_ISO7380_Pad, MountingHole:MountingHole_3.2mm_M3_ISO7380_Pad, F.Cu at (159.5, 50.5)
- added H3: MountingHole_3.2mm_M3_ISO7380_Pad, MountingHole:MountingHole_3.2mm_M3_ISO7380_Pad, F.Cu at (69.5, 138.5)
- added H4: MountingHole_3.2mm_M3_ISO7380_Pad, MountingHole:MountingHole_3.2mm_M3_ISO7380_Pad, F.Cu at (159.5, 138.5)
- C1: footprint Capacitor_SMD:C_0402_1005Metric -> Capacitor_SMD:C_0805_2012Metric
- D1: footprint Diode_SMD:D_0805_2012Metric -> Diode_SMD:D_SOD-123
- R1: value 68R -> 33R; footprint Resistor_SMD:R_0402_1005Metric -> Resistor_SMD:R_0805_2012Metric
- R2, R4: footprint Resistor_SMD:R_0402_1005Metric -> Resistor_SMD:R_0805_2012Metric
- R5: value 280R -> 270R; footprint Resistor_SMD:R_0402_1005Metric -> Resistor_SMD:R_0805_2012Metric
- moved R1 16.7 mm to (78.2, 126.5), turned to -90 degrees
- moved R2 15.3 mm to (82.5, 126.5), turned to 90 degrees
- moved D1 7.16 mm to (96.0, 121.0), turned to 90 degrees
- moved R5 2.79 mm to (106.9, 122.7)
- moved R4 2.74 mm to (100.3, 122.7)
- moved U1 1.39 mm to (103.7, 113.7), turned to -90 degrees
- moved U2 0.48 mm to (140.4, 119.0)
Connections:
- J2 pad 2: unconnected-(J2-Pad2) -> Net-(R2-Pad1)
- J2 pad 4: Net-(J2-Pad4) -> unconnected-(J2-Pad4)
- R2 pad 1: Net-(J2-Pad4) -> Net-(R2-Pad1)
Routing:
- net Net-(J2-Pad4): track 23.3 -> 0.00 mm
- net Net-(R1-Pad2): track 33.7 -> 13.5 mm
- net +3V3: track 125.9 -> 142.8 mm
- net /SCL1: track 115.0 -> 99.4 mm
- net /Rx: track 65.3 -> 55.4 mm
- net Net-(D1-Pad1): track 9.32 -> 18.6 mm
- net Net-(D1-Pad2): track 21.3 -> 30.4 mm
- net /LED_2: track 101.3 -> 110.1 mm
- net /LED_1: track 97.6 -> 106.2 mm
- net Net-(R2-Pad1): track 0.00 -> 7.94 mm
- net /LED_6: track 80.6 -> 75.9 mm
- net /SDA1: track 104.3 -> 100.2 mm
- net /Tx: track 72.5 -> 76.2 mm
- net /SCL2: track 79.8 -> 82.0 mm
- net /SDA2: track 76.3 -> 77.1 mm
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